Commit message: Added config for world

File: ur_moveit_config/srdf/ur.srdf.xacro (robot description, xacro)
@@ -6,4 +6,14 @@
   <xacro:arg name="prefix" default="" />
   <xacro:include filename="$(find ur_moveit_config)/srdf/ur_macro.srdf.xacro"/>
+  <disable_collisions link1="slider_base" link2="base_link_inertia" reason="Adjacent" />
+  <disable_collisions link1="slider_base" link2="base_link" reason="Adjacent" />
+  <disable_collisions link1="slider_base" link2="linear_rail" reason="Adjacent" />
+  <disable_collisions link1="base_link" link2="linear_rail" reason="Adjacent" />
+  <disable_collisions link1="base_link" link2="linear_rail" reason="Adjacent" />
+  <disable_collisions link1="base_link" link2="linear_rail" reason="Adjacent" />
+  <disable_collisions link1="table1" link2="work_cell" reason="Adjacent" />
+  <disable_collisions link1="table2" link2="work_cell" reason="Adjacent" />
+  <disable_collisions link1="linear_rail" link2="work_cell" reason="Adjacent" />
+  <disable_collisions link1="plc_linear_rail" link2="work_cell" reason="Adjacent" />
   <xacro:ur_srdf name="$(arg name)" prefix="$(arg prefix)"/>
 </robot>

File: ur_moveit_config/srdf/ur_macro.srdf.xacro (robot description, xacro)
@@ -12,5 +12,5 @@
     <!--SUBGROUPS - Groups can also be formed by referencing to already defined group names-->
     <group name="${prefix}${name}_manipulator">
-      <chain base_link="${prefix}base_link" tip_link="${prefix}tool0" />
+      <chain base_link="${prefix}base_link" tip_link="${prefix}hex_qc_ft_sensor" />
     </group>
     <!--GROUP STATES - Purpose - Define a named state for a particular group, in terms of joint values. This is useful to define states like 'folded arms'-->
@@ -18,24 +18,16 @@
       <joint name="${prefix}elbow_joint" value="0" />
       <joint name="${prefix}shoulder_lift_joint" value="-1.5707" />
-      <joint name="${prefix}shoulder_pan_joint" value="0" />
-      <joint name="${prefix}wrist_1_joint" value="0" />
-      <joint name="${prefix}wrist_2_joint" value="0" />
-      <joint name="${prefix}wrist_3_joint" value="0" />
-    </group_state>
-    <group_state name="${prefix}up" group="${prefix}${name}_manipulator">
-      <joint name="${prefix}elbow_joint" value="0" />
-      <joint name="${prefix}shoulder_lift_joint" value="-1.5707" />
-      <joint name="${prefix}shoulder_pan_joint" value="0" />
+      <joint name="${prefix}shoulder_pan_joint" value="-0.7854" />
       <joint name="${prefix}wrist_1_joint" value="-1.5707" />
       <joint name="${prefix}wrist_2_joint" value="0" />
       <joint name="${prefix}wrist_3_joint" value="0" />
     </group_state>
-    <group_state name="${prefix}test_configuration" group="${prefix}${name}_manipulator">
-      <joint name="${prefix}elbow_joint" value="1.4" />
-      <joint name="${prefix}shoulder_lift_joint" value="-1.62" />
-      <joint name="${prefix}shoulder_pan_joint" value="1.54" />
-      <joint name="${prefix}wrist_1_joint" value="-1.2" />
-      <joint name="${prefix}wrist_2_joint" value="-1.6" />
-      <joint name="${prefix}wrist_3_joint" value="-0.11" />
+    <group_state name="${prefix}elbow_up" group="${prefix}${name}_manipulator">
+      <joint name="${prefix}elbow_joint" value="1.1868" />
+      <joint name="${prefix}shoulder_lift_joint" value="-0.925" />
+      <joint name="${prefix}shoulder_pan_joint" value="0.7853" />
+      <joint name="${prefix}wrist_1_joint" value="-1.8326" />
+      <joint name="${prefix}wrist_2_joint" value="-1.5707" />
+      <joint name="${prefix}wrist_3_joint" value="0" />
     </group_state>
     <!--END EFFECTOR - Purpose - Represent information about an end effector.-->
@@ -47,4 +39,6 @@
     <disable_collisions link1="${prefix}tool0" link2="${prefix}wrist_2_link" reason="Never" />
     <disable_collisions link1="${prefix}tool0" link2="${prefix}wrist_3_link" reason="Adjacent" />
+    <disable_collisions link1="${prefix}tool0" link2="${prefix}hex_qc_ft_sensor" reason="Adjacent" />
+    <disable_collisions link1="${prefix}wrist_3_link" link2="${prefix}hex_qc_ft_sensor" reason="Adjacent" />
     <disable_collisions link1="${prefix}forearm_link" link2="${prefix}upper_arm_link" reason="Adjacent" />
     <disable_collisions link1="${prefix}forearm_link" link2="${prefix}wrist_1_link" reason="Adjacent" />
